File: pcb/ottawa-badges-2016.kicad_pcb (KiCad board)
At the start: 2 copper layers, 49 x 100 mm, 105 parts, among them P1 USB_OTG, P10 CONN_01X01, P2 CONN_01X08, P3 CONN_01X06, P4 CONN_01X10, P5 CONN_01X08, P6 CONN_02X03, P7 CONN_01X01, P8 CONN_01X01, P9 CONN_01X04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

Commit message: Adding all latest files.
Parts:
- removed the G*** at (74.5, 146.0)
- removed the G*** at (74.5, 98.0)
- removed P7, P8: CONN_01X01, Mounting_Holes:MountingHole_4mm_Pad_Via
- added J1: Conn_01x03, Pin_Headers:Pin_Header_Straight_1x03_Pitch2.54mm, B.Cu at (74.5, 107.0)
- added J2: Conn_02x02_Odd_Even, Pin_Headers:Pin_Header_Straight_2x02_Pitch2.54mm, F.Cu at (52.5, 110.0)
- added J3: Conn_02x02_Odd_Even, Pin_Headers:Pin_Header_Straight_2x02_Pitch2.54mm, F.Cu at (94.0, 110.0)
- added R18: 470, Resistors_SMD:R_0603, B.Cu at (77.5, 107.0)
- added R19: 470, Resistors_SMD:R_0603, B.Cu at (77.5, 104.5)
- added R20: 470, Resistors_SMD:R_0603, F.Cu at (77.8, 107.0)
- added R21: 470, Resistors_SMD:R_0603, F.Cu at (77.8, 104.4)
- moved REF** 7.02 mm to (78.5, 116.8)
- moved C1 5.95 mm to (81.0, 98.6)
- moved C6 1.70 mm to (79.2, 98.6), turned to 270 degrees
Connections:
- JP8 pad 1: /ANALOG4 -> /DIGITAL11
- P1 pad 4: Net-(P1-Pad4) -> (no net)
- P2 pad 1: Net-(P2-Pad1) -> (no net)
- P2 pad 8: Net-(P2-Pad8) -> (no net)
- U2 pad 4: Net-(U2-Pad4) -> (no net)
Routing:
- net /DIGITAL1: track 96.3 -> 19.4 mm, vias 2 -> 0
- net /ANALOG5: track 87.0 -> 140.3 mm, vias 3 -> 5
- net /DIGITAL11: track 47.5 -> 90.5 mm, vias 1 -> 2
- net GND: track 466.0 -> 498.1 mm, vias 8 -> 7
- net /ANALOG4: track 113.4 -> 142.4 mm, vias 3 -> 4
- net +3V3: track 158.6 -> 185.0 mm
- net /DIGITAL0: track 45.2 -> 21.5 mm
- net /PE3: track 16.4 -> 29.4 mm
- net /PE2: track 17.2 -> 28.1 mm
- net /AREF: track 51.2 -> 43.1 mm
- net Net-(J1-Pad2): track 0.00 -> 4.84 mm
- net Net-(J1-Pad1): track 0.00 -> 4.80 mm
- net Net-(D1-Pad1): track 63.2 -> 64.7 mm
Other:
- board text added: "2018 Maker"
- board text added: "CR2032 battery, + side towards metal bracket"
- board text added: "Emergency Resistors Use only in case of scheduling snafu"
- board text added: "To download code to this badge, and for more details on how it works, please visit: https://github.com/rglenn/ottawa-badges-2018/wiki"
- board text removed: "2016 Maker"
- board text removed: "Assembly by"
- board text removed: "DIGITAL0"
- board text removed: "DIGITAL1"
- board text removed: "Replace with CR2032 battery, + side towards metal bracket"
- board text removed: "To download code to this badge, and for more details on how it works, please visit: https://github.com/rglenn/ottawa-badges-2016/wiki"
