File: pcb/ottawa-badges-2016.sch (KiCad schematic (older format))
At the start: 96 parts, among them P1 USB_OTG, P10 CONN_01X01, P2 CONN_01X08, P3 CONN_01X06, P4 CONN_01X10, P5 CONN_01X08, P6 CONN_02X03, P7 CONN_01X01, P8 CONN_01X01, P9 CONN_01X04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

Commit message: Adding all latest files.
Parts:
- removed P7, P8: CONN_01X01, Mounting_Holes:MountingHole_4mm_Pad_Via, symbol CONN_01X01
- added J1: Conn_01x03, Pin_Headers:Pin_Header_Straight_1x03_Pitch2.54mm, symbol Conn_01x03
- added J2, J3: Conn_02x02_Odd_Even, Pin_Headers:Pin_Header_Straight_2x02_Pitch2.54mm, symbol Conn_02x02_Odd_Even
- added R18, R19, R20, R21: 470, Resistors_SMD:R_0603, symbol R
Connections:
- net +3V3: now also J2.1 (Pin_1), J3.1 (Pin_1), R18.2, R19.2
- net ANALOG4: now also J2.2 (Pin_2), J3.2 (Pin_2); no longer JP8.1
- net ANALOG5: now also J2.4 (Pin_4), J3.4 (Pin_4)
- net DIGITAL11: now also JP8.1
- net GND: now also J1.3 (Pin_3), J2.3 (Pin_3), J3.3 (Pin_3)
- net PE2: now also R21.2
- net PE3: now also R20.2
- new net: J1.1 (Pin_1), R18.1, R20.1
- new net: J1.2 (Pin_2), R19.1, R21.1
